File: M0_v1.0.brd (EAGLE design)
At the start: 68.6 x 53.3 mm, 61 parts, among them CN1 POWER_JACK, CN2 47346-0001, CN3 DIGITAL10, CN4 DIGITAL8, CN5 ICSP, CN6 POWER8, CN7 ANALOG6, CN8 SWD, CN9 UART, IC1 AMS1117-5.0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

Commit message: Redone routing of the board
Parts:
- moved C17 20.4 mm to (55.5, 39.6), turned to 135 degrees
- moved C8 9.63 mm to (40.7, 28.2), turned to 45 degrees
- moved C15 7.71 mm to (55.0, 38.0), turned to 135 degrees
- moved C14 7.21 mm to (42.4, 35.5), turned to 45 degrees
- moved R3 6.93 mm to (41.5, 26.6), turned to 315 degrees
- moved C9 6.84 mm to (58.2, 27.6), turned to 315 degrees
- moved R12 6.45 mm to (42.9, 25.2), turned to 315 degrees
- moved L3 6.20 mm to (57.2, 26.6), turned to 315 degrees
- moved C19 5.74 mm to (56.2, 25.6), turned to 135 degrees
- moved Q2 5.26 mm to (51.0, 22.7), turned to 225 degrees
- moved C7 5.21 mm to (43.4, 26.7), turned to 135 degrees
- moved R6 4.98 mm to (42.8, 29.3), turned to 315 degrees
- moved C12 4.27 mm to (49.1, 23.9), turned to 45 degrees
- moved C16 4.23 mm to (44.4, 27.7), turned to 135 degrees
- moved C13 4.02 mm to (52.4, 24.9), turned to 135 degrees
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Routing:
- net SPI_MOSI: track 40.7 -> 19.9 mm, vias 3 -> 1
- net SPI_MISO: track 36.2 -> 18.4 mm, vias 3 -> 1
- net SPI_SCK: track 36.3 -> 18.7 mm, vias 3 -> 1
- net UART_RX: track 46.2 -> 29.8 mm
- net RESET: track 128.0 -> 114.6 mm, vias 4 -> 3
- net UART_TX: track 42.8 -> 29.5 mm
- net 5V: track 103.2 -> 115.0 mm, vias 4 -> 3
- net D13_SCK: track 66.6 -> 78.4 mm, vias 2 -> 3
- net A4: track 46.9 -> 35.2 mm, vias 1 -> 0
- net 3.3V: track 188.2 -> 176.7 mm, vias 13 -> 12
- net D2: track 28.7 -> 17.2 mm, vias 2 -> 0
- net D7: track 28.1 -> 16.8 mm, vias 2 -> 1
- net D6_PWM: track 28.1 -> 16.9 mm, vias 2 -> 1
- net RX_LED: track 62.8 -> 52.4 mm
- net A3: track 45.8 -> 35.8 mm, vias 1 -> 0
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
Commit message: Moved some traces around. Updates some texts.
Parts:
- U1: value ATSAMD21G-AU -> ATSAMD21G18A-AU
- U2: value ATSAMD21G-MU -> ATSAMD21G18A-MU
Routing:
- net D11_MOSI: track 21.0 -> 23.1 mm, vias 1 -> 0
- net GND: track 124.3 -> 125.4 mm, vias 220 -> 235
- net SDA: track 32.5 -> 31.6 mm
- net D10_SS: track 20.7 -> 19.9 mm
Other:
- board text added: "D21G18"
- board text added: "M0/D21G18 v1.0 (c) Andriy Golovnya Designed in Germany http://redscorp.net"
- board text removed: "M0 v1.0 (c) Andriy Golovnya Designed in Germany http://redscorp.net"

Commit message: Moved some traces around
Parts:
- moved C19 0.40 mm to (56.0, 25.2), turned to 315 degrees
- moved C9 0.28 mm to (58.5, 27.7)
Routing:
- net AREF: track 63.5 -> 58.7 mm
- net GND: track 125.4 -> 128.3 mm, vias 235 -> 253

Commit message: Added tooling holes for JLCPCB.
Parts:
- added HOLE1, HOLE2, HOLE3: TOOLINGHOLE, _my_fiducia:TOOLING-HOLE
Changed lines of the file:
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@@
 <attribute name="VALUE" x="58.818665625" y="28.219659375" size="0.6096" layer="27" font="vector" rot="R315"/>
 </element>
+<element name="HOLE1" library="_my_fiducia" package="TOOLING-HOLE" value="TOOLINGHOLE" x="6.35" y="49.403" smashed="yes"/>
+<element name="HOLE2" library="_my_fiducia" package="TOOLING-HOLE" value="TOOLINGHOLE" x="3.048" y="4.826" smashed="yes"/>
+<element name="HOLE3" library="_my_fiducia" package="TOOLING-HOLE" value="TOOLINGHOLE" x="65.913" y="11.938" smashed="yes"/>
 </elements>
 <signals>
@@
 <via x="5.969" y="35.433" extent="1-16" drill="0.35"/>
 <via x="12.192" y="48.768" extent="1-16" drill="0.35"/>
-<via x="6.35" y="48.641" extent="1-16" drill="0.35"/>
+<via x="4.572" y="49.149" extent="1-16" drill="0.35"/>
 <via x="1.397" y="52.197" extent="1-16" drill="0.35"/>
 <via x="22.352" y="4.064" extent="1-16" drill="0.35"/>
